File: mxr phase 45.kicad_pcb (KiCad board)
At the start: 2 copper layers, 58 x 75.5 mm, 42 parts, among them Q2 Q_NJFET_DSG, Q3 Q_NJFET_DSG, Q5 2N3906, U1 TL072, U2 TL072

Commit message: fix
Other:
- board text added: "Phaser 45 ¯\_(ツ)_/¯"
- board text removed: "Phaser 45 ¯\_(ツ)_/¯ Juho & Maksim"
Changed lines of the file:
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@@
 	)
 	(gr_rect
-		(start 151 59.825)
+		(start 151.5 59.825)
 		(end 155 76.325)
 		(stroke
@@
 		)
 	)
-	(gr_text "Phaser 45 ¯\\_(ツ)_/¯\nJuho & Maksim"
+	(gr_text "Phaser 45 ¯\\_(ツ)_/¯"
 		(at 154.5 75.825 90)
 		(layer "F.SilkS")
